File: avr328usbc.kicad_pcb (KiCad board)
At the start: 2 copper layers, 23 parts, among them J1 USB-C THT, J2 MCP Debug Header, J3 USB-C THT, J4 Conn_01x14_MountingPin, J5 AVR-ISP-6, J6 Conn_01x14_MountingPin, J7 MCP Debug Header, U1 MCP2221AxP, U2 ACPL-772L-000E, U3 ACPL-772L-000E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

Commit message: much of board routed
Parts:
- moved J5 6.25 mm to (111.8, 67.9), turned to 0 degrees
Routing:
- net VCC_AVR: track 13.8 -> 145.1 mm
- net VCC_USB: track 8.56 -> 96.0 mm
- net /MCU Sheet/PB3: track 0.00 -> 74.1 mm
- net /MCU Sheet/PB4: track 0.00 -> 73.0 mm, vias 0 -> 1
- net /MCU Sheet/PB5: track 0.00 -> 70.3 mm
- net /UART_Tx: track 0.00 -> 29.6 mm
- net /MCU Sheet/PC6 #RESET: track 0.00 -> 19.9 mm
- net /UART_Rx: track 0.00 -> 19.5 mm
- net /D+: track 0.00 -> 14.4 mm
- net /D-: track 0.00 -> 14.1 mm
- net /MCP.UTx: track 0.00 -> 12.0 mm
- net /MCP.URx: track 0.00 -> 12.0 mm
- net /MCU Sheet/PC5: track 0.00 -> 7.37 mm
- net /MCU Sheet/PC4: track 0.00 -> 7.37 mm
- net /MCU Sheet/PC3: track 0.00 -> 7.37 mm
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
Commit message: first pass at ground plane
Routing:
- net GND_AVR: track 4.57 -> 0.00 mm
- added copper zone on B.Cu, net GND_AVR
- added copper zone on B.Cu, net GND_USB
Other:
- board outline added: 73.3 x 45 mm
Changed lines of the file:
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@@
 		(layer "Dwgs.User")
+	)
+	(gr_rect
+		(start 76.2 63.754)
+		(end 149.479 108.712)
+		(locked yes)
+		(stroke
+			(width 0.05)
+			(type default)
+		)
+		(fill none)
+		(layer "Edge.Cuts")
 	)
 	(segment
@@
 		(layer "B.Cu")
 		(net 2)
-	)
-	(segment
-		(start 125.984 90.424)
-		(end 130.556 90.424)
-		(width 0.2032)
-		(layer "F.Cu")
-		(net 3)
 	)
 	(segment
@@
 		(net 53)
 	)
+	(zone
+		(net 1)
+		(net_name "GND_USB")
+		(locked yes)
+		(layer "B.Cu")
+		(name "USB_GND")
+		(hatch edge 0.5)
+		(connect_pads
+			(clearance 0.5)
+		)
+		(min_thickness 0.25)
+		(filled_areas_thickness no)
+		(fill yes
+			(thermal_gap 0.5)
+			(thermal_bridge_width 0.5)
+		)
+		(polygon
+			(pts
+				(xy 76.962 107.95) (xy 76.962 79.756) (xy 113.03 79.756) (xy 113.03 107.95)
+			)
+		)
+	)
+	(zone
+		(net 3)
+		(net_name "GND_AVR")
+		(locked yes)
+		(layer "B.Cu")
+		(name "AVR_GND")
+		(hatch edge 0.5)
+		(priority 1)
+		(connect_pads
+			(clearance 0.5)
+		)
+		(min_thickness 0.25)
+		(filled_areas_thickness no)
+		(fill yes
+			(thermal_gap 0.5)
+			(thermal_bridge_width 0.5)
+		)
+		(polygon
+			(pts
+				(xy 76.962 79.121) (xy 76.962 64.516) (xy 148.971 64.516) (xy 148.971 108.077) (xy 113.665 107.95)
+				(xy 113.665 79.121)
+			)
+		)
+	)
 )

Commit message: after first look at DRC
Routing:
- net GND_AVR: track 0.00 -> 2.70 mm
- net GND_USB: track 0.00 -> 2.70 mm
Changed lines of the file:
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@@
+	)
+	(segment
+		(start 82.303596 94.121754)
+		(end 80.953596 94.121754)
+		(width 0.508)
+		(layer "B.Cu")
+		(net 1)
+	)
+	(segment
+		(start 80.953596 100.071754)
+		(end 82.303596 100.071754)
+		(width 0.508)
+		(layer "B.Cu")
+		(net 1)
 	)
 	(segment
@@
 	)
 	(segment
+		(start 80.951145 72.334274)
+		(end 82.301145 72.334274)
+		(width 0.508)
+		(layer "B.Cu")
+		(net 3)
+	)
+	(segment
+		(start 80.951145 66.384274)
+		(end 82.301145 66.384274)
+		(width 0.508)
+		(layer "B.Cu")
+		(net 3)
+	)
+	(segment
