File: avr328usbc.kicad_pcb (KiCad board)
At the start: 2 copper layers, 73.3 x 45 mm, 23 parts, among them J1 USB-C THT, J2 MCP Debug Header, J3 USB-C THT, J4 Conn_01x14_MountingPin, J5 AVR-ISP-6, J6 Conn_01x14_MountingPin, J7 MCP Debug Header, U1 MCP2221AxP, U2 ACPL-772L-000E, U3 ACPL-772L-000E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

Commit message: Added silk text to board
Other:
- board text added: "HugonLabs 2024-03-28"
- board text added: "USB-C Isolator ATmega328 v1.0"
Changed lines of the file:
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@@
 	)
 	(footprint "AAAA_Project_Library:USB_C_Receptacle_GCT_USB4085_Reduced_Pad_Size"
+		(locked yes)
 		(layer "F.Cu")
 		(at 82.301145 66.384274 -90)
@@
 	)
 	(footprint "AAAA_Project_Library:USB_C_Receptacle_GCT_USB4085_Reduced_Pad_Size"
+		(locked yes)
 		(layer "F.Cu")
 		(at 82.303596 94.121754 -90)
@@
 		(layer "Edge.Cuts")
 	)
+	(gr_text "HugonLabs\n2024-03-28"
+		(at 107.696 75.565 0)
+		(layer "B.SilkS")
+		(effects
+			(font
+				(size 1 1)
+				(thickness 0.1)
+			)
+			(justify left bottom mirror)
+		)
+	)
+	(gr_text "USB-C Isolator ATmega328 v1.0"
+		(at 142.748 67.183 0)
+		(layer "B.SilkS")
+		(effects
+			(font
+				(size 1 1)
+				(thickness 0.1)
+			)
+			(justify left bottom mirror)
+		)
+	)
+	(gr_text "USB-C Isolator ATmega328 v1.0"
+		(at 117.221 67.31 0)
+		(layer "F.SilkS")
+		(effects
+			(font
+				(size 1 1)
+				(thickness 0.1)
+			)
+			(justify left bottom)
+		)
+	)
+	(gr_text "HugonLabs\n2024-03-28"
+		(at 91.567 80.264 0)
+		(layer "F.SilkS")
+		(effects
+			(font
+				(size 1 1)
+				(thickness 0.1)
+			)
+			(justify left bottom)
+		)
+	)
 	(segment
