File: avr328usbc.kicad_sch (KiCad schematic)
At the start: 19 parts, among them J1 USB-C THT, J2 MCP Debug Header, J3 USB-C THT, J7 MCP Debug Header, U1 MCP2221AxP, U2 ACPL-772L-000E, U3 ACPL-772L-000E

Commit message: Finished and exported BOM
Parts:
- J2, J7: MFR Part Num 825433-7 -> 9-146280-0; now not fitted
Changed lines of the file:
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@@
 		(in_bom yes)
 		(on_board yes)
-		(dnp no)
+		(dnp yes)
 		(fields_autoplaced yes)
 		(property "Reference" "J2"
@@
 			)
 		)
-		(property "MFR Part Num" "825433-7"
+		(property "MFR Part Num" "9-146280-0"
 			(at 45.72 125.73 0)
 			(effects
@@
 		(in_bom yes)
 		(on_board yes)
-		(dnp no)
+		(dnp yes)
 		(fields_autoplaced yes)
 		(property "Reference" "J7"
@@
 			)
 		)
-		(property "MFR Part Num" "825433-7"
+		(property "MFR Part Num" "9-146280-0"
 			(at 95.25 125.73 0)
 			(effects
