File: untitled.kicad_sch (KiCad schematic)
At the start: 4 parts, among them J4 Conn_01x14_MountingPin, J5 AVR-ISP-6, J6 Conn_01x14_MountingPin, U4 ATmega328P-P

Commit message: Finished and exported BOM
Parts:
- J4, J6: MFR (none) -> TE Connectivity; MFR Part Num (none) -> 9-146280-0; now not fitted
- J5: MFR Amphenol -> Molex; MFR Part Num (none) -> TE Connectivity
Changed lines of the file:
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@@
 		(in_bom yes)
 		(on_board yes)
-		(dnp no)
+		(dnp yes)
 		(fields_autoplaced yes)
 		(property "Reference" "J6"
@@
 		)
 		(property "Description" "Generic connector, single row, 01x14, script generated (kicad-library-utils/schlib/autogen/connector/)"
+			(at 223.52 74.93 0)
+			(effects
+				(font
+					(size 1.27 1.27)
+				)
+				(hide yes)
+			)
+		)
+		(property "MFR" "TE Connectivity"
+			(at 223.52 74.93 0)
+			(effects
+				(font
+					(size 1.27 1.27)
+				)
+				(hide yes)
+			)
+		)
+		(property "MFR Part Num" "9-146280-0"
 			(at 223.52 74.93 0)
 			(effects
@@
 		(in_bom yes)
 		(on_board yes)
-		(dnp no)
+		(dnp yes)
 		(fields_autoplaced yes)
 		(property "Reference" "J4"
@@
 		)
 		(property "Description" "Generic connector, single row, 01x14, script generated (kicad-library-utils/schlib/autogen/connector/)"
+			(at 138.43 73.66 0)
+			(effects
+				(font
+					(size 1.27 1.27)
+				)
+				(hide yes)
+			)
+		)
+		(property "MFR" "TE Connectivity"
+			(at 138.43 73.66 0)
+			(effects
+				(font
+					(size 1.27 1.27)
+				)
+				(hide yes)
+			)
+		)
+		(property "MFR Part Num" "9-146280-0"
 			(at 138.43 73.66 0)
 			(effects
@@
 			)
 		)
-		(property "MFR" "Amphenol"
+		(property "MFR" "Molex"
 			(at 173.99 101.6 0)
 			(effects
@@
 			)
 		)
-		(property "MFR Part Num" ""
+		(property "MFR Part Num" "TE Connectivity"
 			(at 173.99 101.6 0)
 			(effects

Commit message: fixed bug in BOM
Parts:
- J5: MFR Part Num TE Connectivity -> 90130-1206
Changed lines of the file:
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@@
 			)
 		)
-		(property "MFR Part Num" "TE Connectivity"
+		(property "MFR Part Num" "90130-1206"
 			(at 173.99 101.6 0)
 			(effects
